File: QFN-68_8x8_P0.4/QFN-68_8x8_P0.4.kicad_pcb (KiCad board)
At the start: 2 copper layers, 25.4 x 91.4 mm, 6 parts, among them J101 Conn_01x36, J102 Conn_01x36, J103 Conn_01x36, J104 Conn_01x36, U101 QFN-68

Commit message: Created SMDIP-16, QFP-48, QFP-32, QFN-80, QFN-68, QFN-64, QFN-60, QFN-56, QFN-48, QFN-36, QFN-28, QFN-20, QFP-32, QFP-48
Parts:
- moved G*** 1.66 mm to (138.4, 85.5)
Routing:
- net /21: vias 0 -> 6
Other:
- board text added: "14"
- board text added: "20"
- board text added: "26"
- board text added: "32"
- board text added: "37"
- board text added: "43"
- board text added: "49"
- board text added: "55"
- board text added: "62"
- board text added: "7"
Changed lines of the file:
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@@
 	(footprint "libraries:LogoSmall"
 		(layer "F.Cu")
-		(at 138.43 87.122)
+		(at 138.43 85.457121)
 		(property "Reference" "G***"
 			(at 0 0 0)
@@
 	)
 	(gr_rect
+		(start 129.42 93.3)
+		(end 131.52 95.3)
+		(stroke
+			(width 0.1)
+			(type solid)
+		)
+		(fill yes)
+		(layer "F.SilkS")
+	)
+	(gr_rect
 		(start 146.067 74.93)
 		(end 151.24 77.59725)
@@
 	)
 	(gr_rect
-		(start 128.443605 129.54)
-		(end 148.411941 157.48)
+		(start 128.443605 142.855)
+		(end 148.411941 156.75)
+		(stroke
+			(width 0.1)
+			(type solid)
+		)
+		(fill yes)
+		(layer "F.SilkS")
+	)
+	(gr_rect
+		(start 130.41 93.3)
+		(end 146.56 112.42)
 		(stroke
 			(width 0.1)
@@
 	)
 	(gr_rect
+		(start 130.375832 126.29)
+		(end 146.474168 158.1)
+		(stroke
+			(width 0.1)
+			(type solid)
+		)
+		(fill yes)
+		(layer "F.SilkS")
+	)
+	(gr_rect
+		(start 128.435832 127.69)
+		(end 148.404168 141.475)
+		(stroke
+			(width 0.1)
+			(type solid)
+		)
+		(fill yes)
+		(layer "F.SilkS")
+	)
+	(gr_rect
 		(start 130.5645 163.81275)
 		(end 146.87125 164.09215)
@@
 	)
 	(gr_rect
-		(start 128.417739 96.52)
-		(end 148.458532 111.76)
+		(start 128.417739 94.66)
+		(end 148.458532 111.01)
 		(stroke
 			(width 0.1)
@@
 		(layer "Edge.Cuts")
 	)
+	(gr_text "62"
+		(at 148.587739 94.012949 0)
+		(layer "F.SilkS" knockout)
+		(effects
+			(font
+				(size 1 1)
+				(thickness 0.2)
+				(bold yes)
+			)
+			(justify right)
+		)
+	)
 	(gr_text "1"
 		(at 128.397 78.74 0)
@@
 		)
 	)
+	(gr_text "7"
+		(at 128.31 94.01 0)
+		(layer "F.SilkS" knockout)
+		(effects
+			(font
+				(size 1 1)
+				(thickness 0.2)
+				(bold yes)
+			)
+			(justify left)
+		)
+	)
+	(gr_text "37"
+		(at 148.51 157.49 0)
+		(layer "F.SilkS" knockout)
+		(effects
+			(font
+				(size 1 1)
+				(thickness 0.2)
+				(bold yes)
+			)
+			(justify right)
+		)
+	)
 	(gr_text "35"
 		(at 148.463 162.56 0)
@@
 		)
 	)
+	(gr_text "43"
+		(at 148.54 142.22 0)
+		(layer "F.SilkS" knockout)
+		(effects
+			(font
+				(size 1 1)
+				(thickness 0.2)
+				(bold yes)
+			)
+			(justify right)
+		)
+	)
 	(gr_text "34"
 		(at 128.397 162.56 0)
@@
 		)
 	)
+	(gr_text "55"
+		(at 148.587739 111.81 0)
+		(layer "F.SilkS" knockout)
+		(effects
+			(font
+				(size 1 1)
+				(thickness 0.2)
+				(bold yes)
+			)
+			(justify right)
+		)
+	)
 	(gr_text "QFN-68\n8x8mm\n0.4mm Pitch"
 		(at 138.43 162.928819 0)
@@
 		)
 	)
+	(gr_text "32"
+		(at 128.364 157.49 0)
+		(layer "F.SilkS" knockout)
+		(effects
+			(font
+				(size 1 1)
+				(thickness 0.2)
+				(bold yes)
+			)
+			(justify left)
+		)
+	)
+	(gr_text "26"
+		(at 128.31 142.24 0)
+		(layer "F.SilkS" knockout)
+		(effects
+			(font
+				(size 1 1)
+				(thickness 0.2)
+				(bold yes)
+			)
+			(justify left)
+		)
+	)
+	(gr_text "49"
+		(at 148.54 127.06 0)
+		(layer "F.SilkS" knockout)
+		(effects
+			(font
+				(size 1 1)
+				(thickness 0.2)
+				(bold yes)
+			)
+			(justify right)
+		)
+	)
 	(gr_text "THERMAL PAD"
 		(at 138.4385 165.146375 0)
@@
 		)
 	)
+	(gr_text "20"
+		(at 128.37 127.01 0)
+		(layer "F.SilkS" knockout)
+		(effects
+			(font
+				(size 1 1)
+				(thickness 0.2)
+				(bold yes)
+			)
+			(justify left)
+		)
+	)
+	(gr_text "14"
+		(at 128.31 111.807051 0)
+		(layer "F.SilkS" knockout)
+		(effects
+			(font
+				(size 1 1)
+				(thickness 0.2)
+				(bold yes)
+			)
+			(justify left)
+		)
+	)
 	(segment
 		(start 127 165.1)
@@
 		(net 22)
 	)
+	(via
+		(at 138.42 78.9)
+		(size 0.6)
+		(drill 0.3)
+		(layers "F.Cu" "B.Cu")
+		(free yes)
+		(net 22)
+	)
+	(via
+		(at 138.432469 125.894139)
+		(size 0.6)
+		(drill 0.3)
+		(layers "F.Cu" "B.Cu")
+		(free yes)
+		(net 22)
+	)
+	(via
+		(at 138.48 112.95)
+		(size 0.6)
+		(drill 0.3)
+		(layers "F.Cu" "B.Cu")
+		(free yes)
+		(net 22)
+	)
+	(via
+		(at 138.42 91.79)
+		(size 0.6)
+		(drill 0.3)
+		(layers "F.Cu" "B.Cu")
+		(free yes)
+		(net 22)
+	)
+	(via
+		(at 138.43 163.49)
+		(size 0.6)
+		(drill 0.3)
+		(layers "F.Cu" "B.Cu")
+		(free yes)
+		(net 22)
+	)
+	(via
+		(at 138.425 142.195)
+		(size 0.6)
+		(drill 0.3)
+		(layers "F.Cu" "B.Cu")
+		(free yes)
+		(net 22)
+	)
